File: Lights_Board.kicad_pcb (KiCad board)
At the start: 2 copper layers, 100 x 100 mm, 70 parts, among them J1 Conn_ARM_JTAG_SWD_10, J10 LED 4, J11 LED 5, J12 LED 6, J13 OD_In, J2 USB_B_Micro, J3 Main Connection, J5 Main Connection, J6 MCU Interface, J7 LED 1, J8 LED 2, J9 LED 3, Q1 AO3400A, Q2 AO3400A, Q3 AO3400A, Q4 AO3400A, Q5 AO3400A, Q6 AO3400A, U1 STM32F072RBTx, U2 TPS2113, U3 TCAN1042xV, U4 AMS1117-5.0, U5 TPS5430DDA, U6 MPU-6050, U7 ADCS747x, U8 ADCS747x

Commit message: Rev2
Parts:
- removed C16: 100nF, Capacitor_SMD:C_0402_1005Metric
- removed C17: 2.2nF, Capacitor_SMD:C_0402_1005Metric
- added C101: 1uF, Capacitor_SMD:C_0402_1005Metric, F.Cu at (143.3, 136.7)
- added C102: 1uF, Capacitor_SMD:C_0402_1005Metric, F.Cu at (134.9, 136.7)
- added C103: 10uF, Capacitor_Tantalum_SMD:CP_EIA-3216-18_Kemet-A, F.Cu at (140.8, 135.8)
- added C104: 10uF, Capacitor_Tantalum_SMD:CP_EIA-3216-18_Kemet-A, F.Cu at (132.3, 135.9)
- added C105: 100nF, Capacitor_SMD:C_0402_1005Metric, F.Cu at (140.9, 130.1)
- added C106: 100nF, Capacitor_SMD:C_0402_1005Metric, F.Cu at (132.5, 130.2)
- U6: value MPU-6050 -> LSM6DS3; footprint Sensor_Motion:InvenSense_QFN-24_4x4mm_P0.5mm -> Package_LGA:LGA-14_3x2.5mm_P0.5mm_LayoutBorder3x4y
- U7, U8: value ADCS747x -> MCP33151; footprint Package_TO_SOT_SMD:SOT-23-6_Handsoldering -> Package_SO:MSOP-10_3x3mm_P0.5mm
- moved D1 8.57 mm to (148.8, 133.9)
- moved R19 6.33 mm to (152.9, 122.9), turned to -90 degrees
- moved C15 6.33 mm to (158.9, 128.3)
- moved D2 6.32 mm to (151.3, 130.7)
- moved R2 6.27 mm to (152.1, 133.3)
- moved R1 6.21 mm to (152.1, 134.9)
- moved U6 4.39 mm to (155.9, 127.6), turned to 0 degrees
- moved C14 4.07 mm to (156.9, 123.5), turned to 180 degrees
- moved U8 3.69 mm to (135.4, 132.3)
- moved R20 2.49 mm to (154.5, 122.9)
- moved U7 2.35 mm to (143.8, 132.3)
- moved D4 0.75 mm to (171.7, 84.8)
Connections:
- U1 pad 20: /Throttle_CS -> unconnected-(U1-Pad20)
- U1 pad 22: /ADC_Data -> /ADC_MISO
- U1 pad 23: /Board_OK -> /ADC_MOSI
- U1 pad 24: unconnected-(U1-Pad24) -> /Throttle_CS
- U1 pad 25: unconnected-(U1-Pad25) -> /Board_OK
- U1 pad 28: /INT_IMU -> /INT1_IMU
- U6 pad 1: GND -> +3V3
- U6 pad 10: Net-(C16-Pad1) -> unconnected-(U6-Pad10)
- U6 pad 11: GND -> unconnected-(U6-Pad11)
- U6 pad 12: /INT_IMU -> +3V3
- U6 pad 13: +3V3 -> /SCL_IMU
- U6 pad 14: (no net) -> /SDA_IMU
- U6 pad 2: (no net) -> +3V3
- U6 pad 3: (no net) -> +3V3
- U6 pad 4: (no net) -> /INT1_IMU
- U6 pad 5: (no net) -> +3V3
- U6 pad 6: unconnected-(U6-Pad6) -> GND
- U6 pad 7: unconnected-(U6-Pad7) -> GND
- U6 pad 9: GND -> unconnected-(U6-Pad9)
- U7 pad 2: GND -> +5V
- U7 pad 4: /ADC_Clk -> GND
- U7 pad 5: /ADC_Data -> GND
- U8 pad 2: GND -> +5V
- U8 pad 4: /ADC_Clk -> GND
- U8 pad 5: /ADC_Data -> GND
Routing:
- net +3V3: track 199.0 -> 242.4 mm, vias 3 -> 8
- net /INT_IMU: track 34.4 -> 0.00 mm, vias 2 -> 0
- net /ADC_Data: track 24.8 -> 0.00 mm
- net /ADC_MOSI: track 0.00 -> 23.0 mm, vias 0 -> 2
- net /ADC_MISO: track 0.00 -> 22.5 mm, vias 0 -> 2
- net /INT1_IMU: track 0.00 -> 14.1 mm
- net +5V: track 175.0 -> 187.6 mm, vias 5 -> 7
- net /Board_OK: track 7.10 -> 15.6 mm
- net /Error: track 7.05 -> 13.3 mm
- net /SDA_IMU: track 16.5 -> 12.7 mm, vias 2 -> 0
- net /Throttle_CS: track 14.6 -> 11.4 mm, vias 2 -> 0
- net Net-(C16-Pad1): track 2.73 -> 0.00 mm
- net /Break: track 6.00 -> 8.11 mm
- net /SCL_IMU: track 16.6 -> 14.6 mm, vias 0 -> 2
- net /Break_CS: track 15.4 -> 13.4 mm
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