File: Lights_Board.kicad_sch (KiCad schematic)
At the start: 70 parts, among them J1 Conn_ARM_JTAG_SWD_10, J10 LED 4, J11 LED 5, J12 LED 6, J13 OD_In, J2 USB_B_Micro, J3 Main Connection, J5 Main Connection, J6 MCU Interface, J7 LED 1, J8 LED 2, J9 LED 3, Q1 AO3400A, Q2 AO3400A, Q3 AO3400A, Q4 AO3400A, Q5 AO3400A, Q6 AO3400A, U1 STM32F072RBTx, U2 TPS2113, U3 TCAN1042xV, U4 AMS1117-5.0, U5 TPS5430DDA, U6 MPU-6050, U7 ADCS747x, U8 ADCS747x

Commit message: Rev2
Parts:
- removed C16: 100nF, Capacitor_SMD:C_0402_1005Metric, symbol Device:C_Small
- removed C17: 2.2nF, Capacitor_SMD:C_0402_1005Metric, symbol Device:C_Small
- removed U6: MPU-6050, Sensor_Motion:InvenSense_QFN-24_4x4mm_P0.5mm, symbol Sensor_Motion:MPU-6050
- removed U7, U8: ADCS747x, Package_TO_SOT_SMD:SOT-23-6_Handsoldering, symbol JohnLib:ADCS747x
- added C101, C102: 1uF, Capacitor_SMD:C_0402_1005Metric, symbol Device:C_Small
- added C103, C104: 10uF, Capacitor_Tantalum_SMD:CP_EIA-3216-18_Kemet-A, symbol Device:C_Polarized_Small_US
- added C105, C106: 100nF, Capacitor_SMD:C_0402_1005Metric, symbol Device:C_Small
- added U6: LSM6DS3, Package_LGA:LGA-14_3x2.5mm_P0.5mm_LayoutBorder3x4y, symbol Sensor_Motion:LSM6DS3
- added U7, U8: MCP33151, Package_SO:MSOP-10_3x3mm_P0.5mm, symbol JohnLib:MCP33151
- C2: LCSC Part (none) -> C307331
- D1: footprint LED_SMD:LED_0805_2012Metric_Castellated -> LED_SMD:LED_0805_2012Metric; LCSC Part C34499 -> C2297
- D2: footprint LED_SMD:LED_0603_1608Metric_Castellated -> LED_SMD:LED_0603_1608Metric
- D3: footprint LED_SMD:LED_0805_2012Metric_Castellated -> LED_SMD:LED_0805_2012Metric
- D4: footprint Diode_SMD:D_SMC -> Diode_SMD:D_SMA
- U4: LCSC Part C347222 -> C6186
Connections:
- net +3V3: now also C105.2, C106.2, U6.1 (SDO/SA0), U6.12 (CS), U6.2 (SDX), U6.3 (SCX), U6.5 (VDDIO), U6.8 (VDD), U7.10 (Dvio), U8.10 (Dvio)
- net +5V: now also C101.1, C102.1, C103.1, C104.1, U7.1 (Vref), U7.2 (Avdd), U8.1 (Vref), U8.2 (Avdd)
- net ADC_Clk: now also U7.8 (SClk), U8.8 (SClk)
- net Board_OK: now also U1.25 (PC5); no longer U1.23 (PA7)
- net Break: now also U8.3 (Ain+)
- net Break_CS: now also U8.6 (CNVST)
- net GND: now also C101.2, C102.2, C103.2, C104.2, C105.1, C106.1, U6.6 (GND), U6.7 (GND), U7.4 (Ain-), U7.5 (Gnd), U8.4 (Ain-), U8.5 (Gnd)
- net SCL_IMU: now also U6.13 (SCL)
- net SDA_IMU: now also U6.14 (SDA)
- net Throttle: now also U7.3 (Ain+)
- net Throttle_CS: now also U1.24 (PC4), U7.6 (CNVST); no longer U1.20 (PA4)
- net ADC_Data renamed ADC_MISO
- net ADC_MISO: now also U7.7 (SDO), U8.7 (SDO)
- net INT_IMU renamed INT1_IMU
- net INT1_IMU: now also U6.4 (INT1)
- new net ADC_MOSI: U1.23 (PA7), U7.9 (SDI), U8.9 (SDI)
- no-connect marks 39 -> 37
Other:
- moved on the sheet: D1, D2, JP3, JP4, Q1, Q2, Q3, Q4, Q5, Q6, R1, R2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

Commit message: Adding automation
Parts:
- C1, C10, C105, C106, C11, C12, C15, C18, C2, C4: LCSC Part C307331 -> (none); LCSC# (none) -> C307331
- C101, C102, C6, C7, C9: LCSC Part C52923 -> (none); LCSC# (none) -> C52923
- C103, C104: LCSC Part C7171 -> (none); LCSC# (none) -> C7171
- C13: LCSC Part C23733 -> (none); LCSC# (none) -> C23733
- C14, C3, C8: LCSC Part C15195 -> (none); LCSC# (none) -> C15195
- C5: LCSC Part C3345 -> (none); LCSC# (none) -> C3345
- D1, D3: LCSC Part C2297 -> (none); LCSC# (none) -> C2297
- D2: LCSC Part C2286 -> (none); LCSC# (none) -> C2286
- D4: LCSC Part C22452 -> (none); LCSC# (none) -> C22452
- L1: LCSC Part C38117 -> (none); LCSC# (none) -> C38117
- Q1, Q2, Q3, Q4, Q5, Q6: LCSC Part C20917 -> (none); LCSC# (none) -> C20917
- R1, R2: LCSC Part C8218 -> (none); LCSC# (none) -> C8218
- R10, R13, R15, R16, R9: LCSC Part C25804 -> (none); LCSC# (none) -> C25804
- R14: LCSC Part C22962 -> (none); LCSC# (none) -> C22962
- R17, R19, R20: LCSC Part C4190 -> (none); LCSC# (none) -> C4190
- R18: LCSC Part C21190 -> (none); LCSC# (none) -> C21190
- R21: LCSC Part C22807 -> (none); LCSC# (none) -> C22807
- U4: LCSC Part C6186 -> (none); LCSC# (none) -> C6186
- U5: LCSC Part C9864 -> (none); LCSC# (none) -> C9864
- U6: LCSC Part C784817 -> (none); LCSC# (none) -> C784817
